File: PowerControl.kicad_pcb (KiCad board)
At the start: 2 copper layers, 80 x 80 mm, 21 parts, among them J1 Conn_01x02, J2 Emergency_stop_switch, J3 Emergency_stop_switch, J4 XT60PB-F, J5 XT60PB-M, Q1 Q_PMOS_GDS, Q2 Q_PMOS_GDS, U1 TLP621, U2 TLV76012DBZR

Commit message: Add board
基本的な設計が終了
Parts:
- added C1: 1000u, Capacitor_THT:CP_Radial_D12.5mm_P5.00mm, F.Cu at (91.4, 86.4)
- added H1: MountingHole, MountingHole:MountingHole_3.2mm_M3, F.Cu at (49.0, 73.0)
- added H2: MountingHole, MountingHole:MountingHole_3.2mm_M3, F.Cu at (49.0, 141.0)
- added H3: MountingHole, MountingHole:MountingHole_3.2mm_M3, F.Cu at (132.0, 141.0)
- added H4: MountingHole, MountingHole:MountingHole_3.2mm_M3, F.Cu at (132.0, 73.0)
- C2, C3: moved to B.Cu
- moved C3 33.8 mm to (90.0, 94.0), turned to 180 degrees
- moved C2 32.8 mm to (90.0, 90.0), turned to 180 degrees
- moved JP1 16.3 mm to (72.0, 93.3)
- moved JP2 16.3 mm to (72.0, 106.0)
- moved JP3 16.3 mm to (72.0, 118.7)
- moved J1 15.6 mm to (76.2, 95.1)
- moved J2 15.6 mm to (76.2, 107.8)
- moved J3 15.6 mm to (76.2, 120.5)
- moved U1 14.8 mm to (88.9, 99.1)
- moved R1 12.9 mm to (86.9, 96.0)
- moved J4 12.4 mm to (96.9, 74.0)
- moved C5 2.81 mm to (88.0, 118.0), turned to 180 degrees
- moved C4 2.24 mm to (89.0, 110.0)
- moved R4 1.10 mm to (93.0, 113.1)
- moved R2 0.80 mm to (93.0, 115.8)
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Routing:
- net Net-(J3-Pad1): track 44.8 -> 27.5 mm
- net /12V: track 33.5 -> 39.3 mm
- net VCC: track 0.00 -> 3.18 mm, vias 3 -> 131
- net Net-(R1-Pad1): track 5.13 -> 3.54 mm
- net Net-(J2-Pad1): track 28.0 -> 27.1 mm
- net Net-(J2-Pad2): track 28.6 -> 28.0 mm
- net GND: track 11.2 -> 11.8 mm
- net OutPut: vias 0 -> 163
- net GNDPWR: vias 1 -> 72
Other:
- board size 80 x 80 mm -> 91 x 76 mm
- board text added: "Designed by TNK."
- board text added: "Emergency stop switch"
- board text added: "GND"
- board text added: "IC Output"
- board text added: "Power controller Version 1.0"
- board text added: "Signal"

Commit message: Update PowerControl.kicad_pcb
Routing:
- net GNDPWR: vias 72 -> 69
Other:
- board text added: "IC Input"
- board text added: "Input"
- board text added: "Output"
- board text added: "https://github.com/picopicodevil/PowerControl.git"
- board text removed: "IC Output"
Changed lines of the file:
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@@
   (general
     (thickness 1.6)
-    (drawings 15)
-    (tracks 423)
+    (drawings 18)
+    (tracks 422)
     (zones 0)
     (modules 26)
@@
     )
   )
-  (gr_text "IC\nOutput" (at 67 94 270) (layer F.SilkS)
+  (gr_text Output (at 101 132) (layer F.SilkS)
+    (effects (font (size 2 2) (thickness 0.3)))
+  )
+  (gr_text Input (at 100 80) (layer F.SilkS)
+    (effects (font (size 2 2) (thickness 0.3)))
+  )
+  (gr_text https://github.com/picopicodevil/PowerControl.git (at 73 143) (layer B.SilkS)
+    (effects (font (size 1 1) (thickness 0.15)) (justify mirror))
+  )
+  (gr_text "IC\nInput" (at 67 94 270) (layer F.SilkS)
     (effects (font (size 1 1) (thickness 0.15)))
   )
@@
     (effects (font (size 1 1) (thickness 0.15)))
   )
-  (gr_text "Designed by TNK." (at 62 142) (layer F.SilkS)
+  (gr_text "Designed by TNK." (at 70 142) (layer F.SilkS)
     (effects (font (size 1 1) (thickness 0.15)))
   )
-  (gr_text "Power controller\nVersion 1.0" (at 62 138) (layer F.SilkS)
+  (gr_text "Power controller\nVersion 1.0" (at 70 138) (layer F.SilkS)
     (effects (font (size 1 1) (thickness 0.15)))
   )
@@
     (effects (font (size 0.8 0.8) (thickness 0.12)))
   )
-  (gr_text Signal (at 82 92) (layer F.SilkS)
+  (gr_text Signal (at 82 93) (layer F.SilkS)
     (effects (font (size 0.8 0.8) (thickness 0.12)))
   )
@@
   (via (at 84 104) (size 0.6) (drill 0.3) (layers F.Cu B.Cu) (net 2))
   (via (at 86 101) (size 0.6) (drill 0.3) (layers F.Cu B.Cu) (net 2))
-  (via (at 78 94) (size 0.6) (drill 0.3) (layers F.Cu B.Cu) (net 2))
   (via (at 78 104) (size 0.6) (drill 0.3) (layers F.Cu B.Cu) (net 2))
   (via (at 73 96) (size 0.6) (drill 0.3) (layers F.Cu B.Cu) (net 2))
@@
   (via (at 84.6 98.8) (size 0.6) (drill 0.3) (layers F.Cu B.Cu) (net 2))
   (via (at 89.2 95.6) (size 0.6) (drill 0.3) (layers F.Cu B.Cu) (net 2))
-  (via (at 84.7 96) (size 0.6) (drill 0.3) (layers F.Cu B.Cu) (net 2))
   (via (at 90 130) (size 0.6) (drill 0.3) (layers F.Cu B.Cu) (net 2))
   (via (at 90 140) (size 0.6) (drill 0.3) (layers F.Cu B.Cu) (net 2))
@@
   (via (at 65 144) (size 0.6) (drill 0.3) (layers F.Cu B.Cu) (net 2))
   (via (at 55 144) (size 0.6) (drill 0.3) (layers F.Cu B.Cu) (net 2))
-  (via (at 82 94) (size 0.6) (drill 0.3) (layers F.Cu B.Cu) (net 2))
   (via (at 125 120) (size 0.6) (drill 0.3) (layers F.Cu B.Cu) (net 3))
   (via (at 115 120) (size 0.6) (drill 0.3) (layers F.Cu B.Cu) (net 3))
@@
   (via (at 130 117) (size 0.6) (drill 0.3) (layers F.Cu B.Cu) (net 3))
   (via (at 91 122) (size 0.6) (drill 0.3) (layers F.Cu B.Cu) (net 3))
-  (segment (start 82.6 92.6) (end 86 96) (width 0.4) (layer F.Cu) (net 4))
-  (segment (start 76.2 92.6) (end 82.6 92.6) (width 0.4) (layer F.Cu) (net 4))
+  (segment (start 82.7 94.5) (end 84.2 96) (width 0.4) (layer F.Cu) (net 4))
+  (segment (start 84.2 96) (end 86 96) (width 0.4) (layer F.Cu) (net 4))
+  (segment (start 76.2 92.6) (end 78.1 94.5) (width 0.4) (layer F.Cu) (net 4))
+  (segment (start 78.1 94.5) (end 82.7 94.5) (width 0.4) (layer F.Cu) (net 4))
   (segment (start 86.36 99.06) (end 82.44 95.14) (width 0.4) (layer F.Cu) (net 5))
   (segment (start 82.44 95.14) (end 76.2 95.14) (width 0.4) (layer F.Cu) (net 5))

Commit message: change Pch MOSFET name
Pch MOSFETの名称をIPD80P03P4L-07に変更
Parts:
- Q1, Q2: value Q_PMOS_GDS -> IPD80P03P4L-07
Changed lines of the file:
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@@
       (effects (font (size 1 1) (thickness 0.15)))
     )
-    (fp_text value Q_PMOS_GDS (at 0 4.5 90) (layer F.Fab)
+    (fp_text value IPD80P03P4L-07 (at 0 4.5 90) (layer F.Fab)
       (effects (font (size 1 1) (thickness 0.15)))
     )
@@
     (tags "solder jumper open")
     (attr virtual)
-    (fp_text reference JP1 (at 0 -1.8 90) (layer F.SilkS)
+    (fp_text reference JP1 (at 0 -1.8 270) (layer F.SilkS)
       (effects (font (size 1 1) (thickness 0.15)))
     )
@@
       (effects (font (size 1 1) (thickness 0.15)))
     )
-    (fp_text value Q_PMOS_GDS (at 0 4.5 90) (layer F.Fab)
+    (fp_text value IPD80P03P4L-07 (at 0 4.5 90) (layer F.Fab)
       (effects (font (size 1 1) (thickness 0.15)))
     )
@@
       (rotate (xyz 0 0 0))
     )
+    (model "C:/Users/yuto/OneDrive/Documents/KiCAD/picopicodevil-kicad-library/XT60.pretty/XT60 Female Connector.STEP"
+      (offset (xyz 3.5 0 7))
+      (scale (xyz 1 1 1))
+      (rotate (xyz -90 0 0))
+    )
   )
   (module Connector_AMASS:AMASS_XT60-F_1x02_P7.20mm_Vertical (layer F.Cu)
@@
       (rotate (xyz 0 0 0))
     )
-  )
+    (model "C:/Users/yuto/OneDrive/Documents/KiCAD/picopicodevil-kicad-library/XT60.pretty/XT60 Male Connector.STEP"
+      (offset (xyz 3.5 0 16))
+      (scale (xyz 1 1 1))
+      (rotate (xyz 90 0 0))
+    )
+  )
