File: PowerControl.sch (KiCad schematic (older format))
At the start: 23 parts, among them J1 Conn_01x02, J2 EMS_SW, J3 EMS_SW, J4 XT60PB-F, J5 XT60PB-M, Q1 IPD80P03P4L-07, Q2 IPD80P03P4L-07, U1 TLP621

Commit message: Update: 導通確認用のLEDを配置
Parts:
- added D1, D2: LED, LED_SMD:LED_0603_1608Metric_Pad1.05x0.95mm_HandSolder, symbol Device:LED
- added R6, R7: R, Resistor_SMD:R_0603_1608Metric_Pad0.98x0.95mm_HandSolder, symbol Device:R
Connections:
- net GNDPWR: now also D1.1 (K), D2.1 (K)
- net OutPut: now also R7.1
- net VCC: now also R6.1
- new net: D1.2 (A), R6.2
- new net: D2.2 (A), R7.2
Other:
- moved on the sheet: C1, C2, C3
Changed lines of the file:
@@
 L power:VCC #PWR05
 U 1 1 5EF0A202
-P 3500 3400
-F 0 "#PWR05" H 3500 3250 50  0001 C CNN
-F 1 "VCC" H 3515 3573 50  0000 C CNN
-F 2 "" H 3500 3400 50  0001 C CNN
-F 3 "" H 3500 3400 50  0001 C CNN
-	1    3500 3400
+P 2850 3500
+F 0 "#PWR05" H 2850 3350 50  0001 C CNN
+F 1 "VCC" H 2865 3673 50  0000 C CNN
+F 2 "" H 2850 3500 50  0001 C CNN
+F 3 "" H 2850 3500 50  0001 C CNN
+	1    2850 3500
 	-1   0    0    1
 $EndComp
@@
 L power:GNDPWR #PWR07
 U 1 1 5EF0AE6D
-P 4000 3400
-F 0 "#PWR07" H 4000 3200 50  0001 C CNN
-F 1 "GNDPWR" H 4004 3246 50  0000 C CNN
-F 2 "" H 4000 3350 50  0001 C CNN
-F 3 "" H 4000 3350 50  0001 C CNN
-	1    4000 3400
+P 3350 3500
+F 0 "#PWR07" H 3350 3300 50  0001 C CNN
+F 1 "GNDPWR" H 3354 3346 50  0000 C CNN
+F 2 "" H 3350 3450 50  0001 C CNN
+F 3 "" H 3350 3450 50  0001 C CNN
+	1    3350 3500
 	1    0    0    -1
 $EndComp
@@
 L power:PWR_FLAG #FLG02
 U 1 1 5EF0B77F
-P 4000 3400
-F 0 "#FLG02" H 4000 3475 50  0001 C CNN
-F 1 "PWR_FLAG" H 4000 3573 50  0000 C CNN
-F 2 "" H 4000 3400 50  0001 C CNN
-F 3 "~" H 4000 3400 50  0001 C CNN
-	1    4000 3400
+P 3350 3500
+F 0 "#FLG02" H 3350 3575 50  0001 C CNN
+F 1 "PWR_FLAG" H 3350 3673 50  0000 C CNN
+F 2 "" H 3350 3500 50  0001 C CNN
+F 3 "~" H 3350 3500 50  0001 C CNN
+	1    3350 3500
 	1    0    0    -1
 $EndComp
@@
 L power:PWR_FLAG #FLG01
 U 1 1 5EF0D9A5
-P 3500 3400
-F 0 "#FLG01" H 3500 3475 50  0001 C CNN
-F 1 "PWR_FLAG" H 3500 3573 50  0000 C CNN
-F 2 "" H 3500 3400 50  0001 C CNN
-F 3 "~" H 3500 3400 50  0001 C CNN
-	1    3500 3400
+P 2850 3500
+F 0 "#FLG01" H 2850 3575 50  0001 C CNN
+F 1 "PWR_FLAG" H 2850 3673 50  0000 C CNN
+F 2 "" H 2850 3500 50  0001 C CNN
+F 3 "~" H 2850 3500 50  0001 C CNN
+	1    2850 3500
 	1    0    0    -1
 $EndComp
@@
 L power:PWR_FLAG #FLG03
 U 1 1 5EF0DEF1
-P 4500 3400
-F 0 "#FLG03" H 4500 3475 50  0001 C CNN
-F 1 "PWR_FLAG" H 4500 3573 50  0000 C CNN
-F 2 "" H 4500 3400 50  0001 C CNN
-F 3 "~" H 4500 3400 50  0001 C CNN
-	1    4500 3400
+P 3850 3500
+F 0 "#FLG03" H 3850 3575 50  0001 C CNN
+F 1 "PWR_FLAG" H 3850 3673 50  0000 C CNN
+F 2 "" H 3850 3500 50  0001 C CNN
+F 3 "~" H 3850 3500 50  0001 C CNN
+	1    3850 3500
 	1    0    0    -1
 $EndComp
@@
 L power:GND #PWR08
 U 1 1 5EF0ACCF
-P 4500 3400
-F 0 "#PWR08" H 4500 3150 50  0001 C CNN
-F 1 "GND" H 4505 3227 50  0000 C CNN
-F 2 "" H 4500 3400 50  0001 C CNN
-F 3 "" H 4500 3400 50  0001 C CNN
-	1    4500 3400
+P 3850 3500
+F 0 "#PWR08" H 3850 3250 50  0001 C CNN
+F 1 "GND" H 3855 3327 50  0000 C CNN
+F 2 "" H 3850 3500 50  0001 C CNN
+F 3 "" H 3850 3500 50  0001 C CNN
+	1    3850 3500
 	1    0    0    -1
 $EndComp
@@
 L Device:CP C1
 U 1 1 5EF5DFD2
-P 1750 3450
-F 0 "C1" H 1868 3496 50  0000 L CNN
-F 1 "1000u" H 1868 3405 50  0000 L CNN
-F 2 "Capacitor_THT:CP_Radial_D12.5mm_P5.00mm" H 1788 3300 50  0001 C CNN
-F 3 "~" H 1750 3450 50  0001 C CNN
-	1    1750 3450
+P 1100 3550
+F 0 "C1" H 1218 3596 50  0000 L CNN
+F 1 "1000u" H 1218 3505 50  0000 L CNN
+F 2 "Capacitor_THT:CP_Radial_D12.5mm_P5.00mm" H 1138 3400 50  0001 C CNN
+F 3 "~" H 1100 3550 50  0001 C CNN
+	1    1100 3550
 	1    0    0    -1
 $EndComp
@@
 L power:VCC #PWR01
 U 1 1 5EF5F512
-P 2200 3300
-F 0 "#PWR01" H 2200 3150 50  0001 C CNN
-F 1 "VCC" H 2215 3473 50  0000 C CNN
-F 2 "" H 2200 3300 50  0001 C CNN
-F 3 "" H 2200 3300 50  0001 C CNN
-	1    2200 3300
+P 1550 3400
+F 0 "#PWR01" H 1550 3250 50  0001 C CNN
+F 1 "VCC" H 1565 3573 50  0000 C CNN
+F 2 "" H 1550 3400 50  0001 C CNN
+F 3 "" H 1550 3400 50  0001 C CNN
+	1    1550 3400
 	1    0    0    -1
 $EndComp
@@
 L Device:C C2
 U 1 1 5EF611D5
-P 2200 3450
-F 0 "C2" H 2315 3496 50  0000 L CNN
-F 1 "10u" H 2315 3405 50  0000 L CNN
-F 2 "Capacitor_SMD:C_0805_2012Metric_Pad1.15x1.40mm_HandSolder" H 2238 3300 50  0001 C CNN
-F 3 "~" H 2200 3450 50  0001 C CNN
-	1    2200 3450
+P 1550 3550
+F 0 "C2" H 1665 3596 50  0000 L CNN
+F 1 "10u" H 1665 3505 50  0000 L CNN
+F 2 "Capacitor_SMD:C_0805_2012Metric_Pad1.15x1.40mm_HandSolder" H 1588 3400 50  0001 C CNN
+F 3 "~" H 1550 3550 50  0001 C CNN
+	1    1550 3550
 	1    0    0    -1
 $EndComp
@@
 L Device:C C3
 U 1 1 5EF62FBC
-P 2600 3450
-F 0 "C3" H 2715 3496 50  0000 L CNN
-F 1 "1u" H 2715 3405 50  0000 L CNN
-F 2 "Capacitor_SMD:C_0805_2012Metric_Pad1.15x1.40mm_HandSolder" H 2638 3300 50  0001 C CNN
-F 3 "~" H 2600 3450 50  0001 C CNN
-	1    2600 3450
-	1    0    0    -1
-$EndComp
-Wire Wire Line
-	2600 3300 2200 3300
-Connection ~ 2200 3300
-Wire Wire Line
-	2200 3300 1750 3300
-Wire Wire Line
-	1750 3600 2200 3600
-Connection ~ 2200 3600
-Wire Wire Line
-	2200 3600 2600 3600
+P 1950 3550
+F 0 "C3" H 2065 3596 50  0000 L CNN
+F 1 "1u" H 2065 3505 50  0000 L CNN
+F 2 "Capacitor_SMD:C_0805_2012Metric_Pad1.15x1.40mm_HandSolder" H 1988 3400 50  0001 C CNN
+F 3 "~" H 1950 3550 50  0001 C CNN
+	1    1950 3550
+	1    0    0    -1
+$EndComp
+Wire Wire Line
+	1950 3400 1550 3400
+Connection ~ 1550 3400
+Wire Wire Line
+	1550 3400 1100 3400
+Wire Wire Line
+	1100 3700 1550 3700
+Connection ~ 1550 3700
+Wire Wire Line
+	1550 3700 1950 3700
 $Comp
 L power:GNDPWR #PWR02
 U 1 1 5EF65C0A
-P 2200 3600
-F 0 "#PWR02" H 2200 3400 50  0001 C CNN
-F 1 "GNDPWR" H 2204 3446 50  0000 C CNN
-F 2 "" H 2200 3550 50  0001 C CNN
-F 3 "" H 2200 3550 50  0001 C CNN
-	1    2200 3600
+P 1550 3700
+F 0 "#PWR02" H 1550 3500 50  0001 C CNN
+F 1 "GNDPWR" H 1554 3546 50  0000 C CNN
+F 2 "" H 1550 3650 50  0001 C CNN
+F 3 "" H 1550 3650 50  0001 C CNN
+	1    1550 3700
 	1    0    0    -1
 $EndComp
@@
 	1    0    0    -1
 $EndComp
+$Comp
+L Device:LED D1
+U 1 1 61464DFE
+P 4550 3800
+F 0 "D1" V 4589 3682 50  0000 R CNN
+F 1 "LED" V 4498 3682 50  0000 R CNN
+F 2 "LED_SMD:LED_0603_1608Metric_Pad1.05x0.95mm_HandSolder" H 4550 3800 50  0001 C CNN
+F 3 "~" H 4550 3800 50  0001 C CNN
+	1    4550 3800
+	0    -1   -1   0
+$EndComp
+$Comp
+L Device:R R6
+U 1 1 614659A6
+P 4550 3500
+F 0 "R6" H 4620 3546 50  0000 L CNN
+F 1 "R" H 4620 3455 50  0000 L CNN
+F 2 "Resistor_SMD:R_0603_1608Metric_Pad0.98x0.95mm_HandSolder" V 4480 3500 50  0001 C CNN
+F 3 "~" H 4550 3500 50  0001 C CNN
+	1    4550 3500
+	1    0    0    -1
+$EndComp
+$Comp
+L Device:LED D2
+U 1 1 6146B713
+P 4950 3800
+F 0 "D2" V 4989 3682 50  0000 R CNN
+F 1 "LED" V 4898 3682 50  0000 R CNN
+F 2 "LED_SMD:LED_0603_1608Metric_Pad1.05x0.95mm_HandSolder" H 4950 3800 50  0001 C CNN
+F 3 "~" H 4950 3800 50  0001 C CNN
+	1    4950 3800
+	0    -1   -1   0
+$EndComp
+$Comp
+L Device:R R7
+U 1 1 6146B719
+P 4950 3500
+F 0 "R7" H 5020 3546 50  0000 L CNN
+F 1 "R" H 5020 3455 50  0000 L CNN
+F 2 "Resistor_SMD:R_0603_1608Metric_Pad0.98x0.95mm_HandSolder" V 4880 3500 50  0001 C CNN
+F 3 "~" H 4950 3500 50  0001 C CNN
+	1    4950 3500
+	1    0    0    -1
+$EndComp
+$Comp
+L power:VCC #PWR0102
+U 1 1 6146D29C
+P 4550 3350
+F 0 "#PWR0102" H 4550 3200 50  0001 C CNN
+F 1 "VCC" H 4565 3523 50  0000 C CNN
+F 2 "" H 4550 3350 50  0001 C CNN
+F 3 "" H 4550 3350 50  0001 C CNN
+	1    4550 3350
+	1    0    0    -1
+$EndComp
+$Comp
+L power:GNDPWR #PWR0103
+U 1 1 6146DF10
+P 4550 3950
+F 0 "#PWR0103" H 4550 3750 50  0001 C CNN
+F 1 "GNDPWR" H 4554 3796 50  0000 C CNN
+F 2 "" H 4550 3900 50  0001 C CNN
+F 3 "" H 4550 3900 50  0001 C CNN
+	1    4550 3950
+	1    0    0    -1
+$EndComp
+Text GLabel 4950 3350 1    50   Input ~ 0
+OutPut
+$Comp
+L power:GNDPWR #PWR0104
+U 1 1 614701AB
+P 4950 3950
+F 0 "#PWR0104" H 4950 3750 50  0001 C CNN
+F 1 "GNDPWR" H 4954 3796 50  0000 C CNN
+F 2 "" H 4950 3900 50  0001 C CNN
+F 3 "" H 4950 3900 50  0001 C CNN
+	1    4950 3950
+	1    0    0    -1
+$EndComp
